File: Hardware/KiCAD/Reverse Engineering - AT90USB162.kicad_sch (KiCad schematic)
At the start: 36 parts, among them J2 ISP Connector, J3 USB A, J4 01x10 Shielded Connector, SW1 SW_DIP_x01, SW2 SW_DIP_x01, SW3 SW_DIP_x01, SW4 SW_DIP_x01, U1 AT90USB162-16A

Commit message: Update
Parts:
- removed SW1, SW2, SW3, SW4: SW_DIP_x01, symbol Switch:SW_DIP_x01
- added SW1, SW2, SW3, SW4: SW_Reed, symbol Switch:SW_Reed
Connections:
- net Earth: now also SW1.2, SW2.2, SW3.2, SW4.2
- net PB4: now also SW1.1
- net PB5: now also SW2.1
- net PB6: now also SW3.1
- net PB7: now also SW4.1
